Commit message: 0729

File: src/ur5/ur5_description/urdf/ur5.urdf.xacro (robot description, xacro)
@@ -81,4 +81,5 @@
     </link>
     <joint name="world_joint" type="fixed">
+        <!-- <origin xyz="0 0 0.025" rpy="0 0 0"/> -->
         <parent link="world"/>
         <child link="${prefix}rail0"/>
@@ -87,5 +88,5 @@
       <parent link="${prefix}rail0"/>
       <child link="${prefix}rail1"/>
-      <origin xyz="0 0 0" rpy="0 0 0"/>
+      <origin xyz="0 0 0.08" rpy="0 0 0"/>
       <axis xyz="0 1 0"/>
       <limit effort="30" velocity="1.0" lower="-2" upper="2"/>
@@ -314,5 +315,5 @@
       <parent link="${prefix}wrist_3_link" />
       <child link = "${prefix}ee_link" />
-      <origin xyz="0.0 ${wrist_3_length} 0.0" rpy="0.0 0.0 ${pi/2.0}" />
+      <origin rpy="${-pi/2} 0 0" xyz="0 0.173 0"/>
     </joint>
     <link name="${prefix}ee_link">
@@ -344,4 +345,32 @@
       <child link="${prefix}tool0"/>
     </joint>
+    <link name="${prefix}_link_knife"/>
+    <joint name="${prefix}_joint_knife" type="fixed">
+        <origin rpy="0 0 0" xyz="0 0.21 0.039"/>
+        <!-- <origin rpy="0 0 0" xyz="0 0.21 0.019"/> -->
+        <parent link="${prefix}ee_link"/>
+        <child link="${prefix}_link_knife"/>
+    </joint>
+    <link name="${prefix}_link_spatula"/>
+    <joint name="${prefix}_joint_spatula" type="fixed">
+        <origin rpy="0 0 0" xyz="0 0.235 0"/>
+        <!-- <origin rpy="0 0 0" xyz="0 0.235 -0.02"/> -->
+        <parent link="${prefix}ee_link"/>
+        <child link="${prefix}_link_spatula"/>
+    </joint>
+    <link name="${prefix}_link_scooper"/>
+    <joint name="${prefix}_joint_scooper" type="fixed">
+        <origin rpy="0 0 0" xyz="0 0.25 0"/>
+        <!-- <origin rpy="0 0 0" xyz="0 0.25 -0.02"/> -->
+        <parent link="${prefix}ee_link"/>
+        <child link="${prefix}_link_scooper"/>
+    </joint>
+    <link name="${prefix}_link_spreader"/>
+    <joint name="${prefix}_joint_spreader" type="fixed">
+        <origin rpy="0 0 0" xyz="0 0.295 -0.002"/>
+        <!-- <origin rpy="0 0 0" xyz="0 0.295 -0.022"/> -->
+        <parent link="${prefix}ee_link"/>
+        <child link="${prefix}_link_spreader"/>
+    </joint>
   </xacro:macro>
 </robot>
